Commit message: feat: Use diff_drive controller. Get parameters from yaml and pass to the urdf

File: urdf/dif_base.urdf.xacro (robot description, xacro)
@@ -1,9 +1,23 @@
 <?xml version="1.0"?>
 <robot xmlns:xacro="http://www.ros.org/wiki/xacro" name="robo_diferenciado">
+    <xacro:arg name="wheel_radius" default="0.1"/>
+    <xacro:arg name="wheel_separation" default="0.175"/>
     <xacro:include filename="$(find robo_diferenciado)/urdf/diferenciado_robot_model.urdf.xacro"/>
     <xacro:include filename="$(find robo_diferenciado)/urdf/wheels.ros2_control.xacro"/>
+    <xacro:robot_diferenciado
+        wheel_radius="$(arg wheel_radius)"
+        wheel_separation="$(arg wheel_separation)"
+        chassis_mass="5.0"
+        chassis_length="0.4"
+        chassis_width="0.3"
+        chassis_height="0.1"
+        wheel_mass="1.0"
+        wheel_width="0.05"
+        caster_radius="0.05"
+        caster_mass="0.5"
+        caster_offset_x="0.15"/>
     <gazebo>
         <plugin filename="gz_ros2_control-system" name="gz_ros2_control::GazeboSimROS2ControlPlugin">
-            <parameters>$(find robo_diferenciado)/config/ros2_control.yaml</parameters>
+            <parameters>$(find robo_diferenciado)/config/diff_drive_control.yaml</parameters>
         </plugin>
     </gazebo>

File: urdf/diferenciado_robot_model.urdf.xacro (robot description, xacro)
@@ -25,14 +25,15 @@
         </inertial>
     </xacro:macro>
-    <xacro:property name="chassis_mass" value="5.0"/>
-    <xacro:property name="chassis_length" value="0.4"/>
-    <xacro:property name="chassis_width" value="0.3"/>
-    <xacro:property name="chassis_height" value="0.1"/>
-    <xacro:property name="wheel_radius" value="0.1"/>
-    <xacro:property name="wheel_width" value="0.05"/>
-    <xacro:property name="wheel_mass" value="1.0"/>
-    <xacro:property name="wheel_offset_y" value="0.175"/> <xacro:property name="caster_radius" value="0.05"/>
-    <xacro:property name="caster_mass" value="0.5"/>
-    <xacro:property name="caster_offset_x" value="0.15"/>
+    <xacro:macro name="robot_diferenciado" params="wheel_radius
+        wheel_separation
+        chassis_mass
+        chassis_length
+        chassis_width
+        chassis_height
+        wheel_mass
+        wheel_width
+        caster_radius
+        caster_mass
+        caster_offset_x">
     <link name="base_link">
     </link>
@@ -81,5 +82,5 @@
         <parent link="chassis"/>
         <child link="left_wheel"/>
-        <origin xyz="-0.1 ${wheel_offset_y} 0" rpy="0 0 0"/> <axis xyz="0 1 0"/>
+        <origin xyz="-0.1 ${wheel_separation} 0" rpy="0 0 0"/> <axis xyz="0 1 0"/>
     </joint>
     <link name="right_wheel">
@@ -104,5 +105,5 @@
         <parent link="chassis"/>
         <child link="right_wheel"/>
-        <origin xyz="-0.1 -${wheel_offset_y} 0" rpy="0 0 0"/> <axis xyz="0 1 0"/>
+        <origin xyz="-0.1 -${wheel_separation} 0" rpy="0 0 0"/> <axis xyz="0 1 0"/>
     </joint>
     <link name="caster_wheel">
@@ -141,3 +142,4 @@
         <material>Gazebo/White</material>
     </gazebo>
+    </xacro:macro>
 </robot>

File: urdf/wheels.ros2_control.xacro (robot description, xacro)
@@ -3,7 +3,5 @@
   <ros2_control name="GazeboSystem" type="system">
     <hardware>
-    	<!-- <plugin>gazebo_ros2_control/GazeboSystem</plugin> -->
 				<plugin>gz_ros2_control/GazeboSimSystem</plugin>
-				<plugin>mock_components/GenericSystem</plugin>
   	</hardware>
     <joint name="left_wheel_joint">
